File: Schematic/Card/Layout.kicad_pcb (KiCad board)
At the start: 2 copper layers, 89 x 51 mm, 28 parts, among them J1 JTAG, J2 Power, U1 RF430FRL

Commit message: Fixed ground issue and cleaned up board
Parts:
- removed G***: LOGO, NFCBusiness:LOGO
- added ?: , NFCBuisness:Name, F.Cu at (170.4, 77.8)
- added ?: , NFCBuisness:Rank, F.Cu at (172.1, 82.4)
- added ?: , NFCBuisness:Bottom, F.Cu at (177.2, 114.7)
- renumbered C2 to C1, C6 to C2, C1 to C3, C5 to C4, C7 to C5, C4 to C6, C3 to C7
Connections:
- U1 pad 25: (no net) -> GND
Routing:
- net GND: track 76.1 -> 80.0 mm, vias 8 -> 9
- net (no net): vias 1 -> 0
Other:
- board text added: "V2a"
- board text removed: "V2"

Commit message: V3, changes may improve reading distance
Parts:
- added C10: 1uF, Capacitors_SMD:C_0805, F.Cu at (137.6, 99.8)
- added R1: 100k, Resistors_SMD:R_0805, F.Cu at (137.6, 103.0)
Connections:
- U1 pad 14: Net-(U1-Pad14) -> GND
- U1 pad 16: Net-(U1-Pad16) -> GND
Routing:
- net Net-(C10-Pad2): track 0.00 -> 8.16 mm
- net Net-(R1-Pad2): track 0.00 -> 4.41 mm
- net GND: track 80.0 -> 82.6 mm, vias 9 -> 12
- net Net-(C1-Pad1): track 17.0 -> 18.6 mm
- net VDDA: track 25.7 -> 24.2 mm
Other:
- board text added: "V3"
- board text removed: "V2a"

Commit message: Added better ground plane
Parts:
- moved Ref** 0.22 mm to (156.0, 98.7)
Routing:
- net GND: vias 12 -> 34
- added copper zone on F.Cu, net GND
Other:
- board text added: "V5"
- board text removed: "V3"
