File: Schematic/2023/NFCBuisnessV3.kicad_pcb (KiCad board)
At the start: 2 copper layers, 87.6 x 49.5 mm, 16 parts, among them J1 Conn_01x01, J2 Conn_01x01, J3 Prog, U1 ST25DV04K-IER8C3, U2 CH32V003FxPx

Commit message: Updated for V2
Parts:
- added C4: C_Small, Capacitor_SMD:C_0805_2012Metric, F.Cu at (130.5, 86.8)
- added C5: C_Small, Capacitor_SMD:C_0805_2012Metric, F.Cu at (130.6, 92.9)
- added J4: Conn_01x03, Connector_PinHeader_2.54mm:PinHeader_1x03_P2.54mm_Vertical, F.Cu at (119.7, 83.7)
- added Y1: Crystal, Crystal:Crystal_SMD_2012-2Pin_2.0x1.2mm_HandSoldering, F.Cu at (131.5, 89.9)
- added kibuzzard-65F9F6C6: G***, kibuzzard-65F9F6C6, B.Cu at (122.2, 87.8)
- U1: footprint Package_DFN_QFN:DFN-8-1EP_3x2mm_P0.5mm_EP1.36x1.46mm -> NFCBuisness:TSSOP_K-IER6T3_STM
- moved kibuzzard-65E89835 5.90 mm to (137.1, 88.9)
- moved U2 5.83 mm to (137.2, 90.4)
- moved J3 5.82 mm to (139.5, 83.6)
- moved C3 1.48 mm to (130.7, 96.3)
- moved R1 1.34 mm to (134.8, 96.3)
- moved C2 0.75 mm to (117.5, 91.7)
- moved U1 0.70 mm to (122.8, 91.9)
Connections:
- U1 pad 5: unconnected-(U1-SDA-Pad5) -> Net-(J4-Pin_1)
- U1 pad 6: unconnected-(U1-SCL-Pad6) -> Net-(J4-Pin_2)
- U1 pad 7: unconnected-(U1-GPO-Pad7) -> Net-(J4-Pin_3)
- U2 pad 5: unconnected-(U2-PA1-Pad5) -> Net-(U2-PA1)
- U2 pad 6: unconnected-(U2-PA2-Pad6) -> Net-(U2-PA2)
Routing:
- net Net-(J4-Pin_1): track 0.00 -> 12.7 mm, vias 0 -> 1
- net Net-(J4-Pin_2): track 0.00 -> 10.9 mm, vias 0 -> 1
- net Net-(J4-Pin_3): track 0.00 -> 9.49 mm, vias 0 -> 1
- net PC1: track 49.2 -> 43.3 mm
- net PC5: track 38.0 -> 32.1 mm
- net PC3: track 23.1 -> 17.3 mm
- net PC4: track 29.8 -> 24.0 mm
- net PC2: track 54.5 -> 48.7 mm
- net PC0: track 41.5 -> 35.7 mm
- net Net-(U2-PA1): track 0.00 -> 5.54 mm
- net Net-(U2-PA2): track 0.00 -> 5.00 mm
- net +3.3V: track 26.5 -> 30.5 mm, vias 2 -> 1
- net VSS: track 43.7 -> 45.3 mm, vias 3 -> 5
- net Net-(D1-K): track 132.5 -> 131.1 mm
- net VCC: track 5.03 -> 3.96 mm, vias 2 -> 0
