File: Schematic/2023/NFCBuisnessV3.kicad_sch (KiCad schematic)
At the start: 15 parts, among them J1 Conn_01x01, J2 Conn_01x01, J3 Prog, U1 ST25DV04K-IER8C3, U2 CH32V003FxPx

Commit message: Updated for V2
Parts:
- added C4, C5: C_Small, Capacitor_SMD:C_0805_2012Metric, symbol Device:C_Small
- added J4: Conn_01x03, Connector_PinHeader_2.54mm:PinHeader_1x03_P2.54mm_Vertical, symbol Connector_Generic:Conn_01x03
- added Y1: Crystal, Crystal:Crystal_SMD_2012-2Pin_2.0x1.2mm_HandSoldering, symbol Device:Crystal
- U1: footprint Package_DFN_QFN:DFN-8-1EP_3x2mm_P0.5mm_EP1.36x1.46mm -> NFCBuisness:TSSOP_K-IER6T3_STM
Connections:
- net VSS: now also C4.2, C5.2
- net at U1.5 (SDA): now also J4.1 (Pin_1)
- net at U1.6 (SCL): now also J4.2 (Pin_2)
- net at U1.7 (GPO): now also J4.3 (Pin_3)
- net at U2.5 (PA1): now also C4.1, Y1.2
- net at U2.6 (PA2): now also C5.1, Y1.1
